Commit message: feat(launch): add listen_only_mode for passive arm mirroring
Adds a listen_only_mode argument, plumbed from launch_params.yaml through
the launch file into the robot ros2_control xacro macro. When enabled, the
arm's ros2_control block is omitted so nothing claims command interfaces
for j1..j6, and joint states are sourced from ros2_forwarder.py talking to
the vendor SDK directly.

Intended for digital-twin use: mirror a physical arm in RViz/Gazebo without
driving it. The forwarder only runs when robot_hardware_connected=true and
listen_only_mode=true, so it can never race FairinoHardwareInterface for the
real connection.

File: src/fairino10_v6_moveit2_config/config/fairino10_v6_robot.ros2_control.xacro (robot description, xacro)
@@ -1,8 +1,9 @@
 <?xml version="1.0"?>
 <robot xmlns:xacro="http://www.ros.org/wiki/xacro">
-    <xacro:macro name="fairino10_v6_robot_ros2_control" params="name initial_positions_file ros2_control_header:=world control_system:=moveit  gripper_name:=none gripper_hardware_connected:=false gripper_hardware_plugin:=none listen_only_mode:=true robot_ip_address:=192.168.58.2">
+    <xacro:macro name="fairino10_v6_robot_ros2_control" params="name initial_positions_file ros2_control_header:=world control_system:=moveit gripper_name:=none gripper_hardware_connected:=false gripper_hardware_plugin:=none listen_only_mode:=true robot_ip_address:=192.168.58.2 ">
         <xacro:property name="initial_positions" value="${xacro.load_yaml(initial_positions_file)['initial_positions']}"/>
         <!-- Xacro arg for control system (Defualted to Rviz/Moveit-->
         <xacro:property name="controllers_yaml_name" value="${'ros2_controllers.yaml' if ros2_control_header == 'world' else 'fairino10_' + ros2_control_header + '_ros2_controllers.yaml'}"/>
+        <xacro:if value="${str(listen_only_mode).lower() == 'false'}">
         <ros2_control name="${name}" type="system">
             <hardware>
@@ -12,5 +13,4 @@
               <xacro:if value="${control_system == 'hardware'}">
                   <plugin>fairino_hardware/FairinoHardwareInterface</plugin>
-                  <param name="robot_ip">${robot_ip_address}</param>
               </xacro:if>
               <xacro:if value="${control_system == 'gazebo'}">
@@ -19,7 +19,5 @@
           </hardware>
           <joint name="j1">
-              <xacro:unless value="${listen_only_mode}">
-                    <command_interface name="position"/>
-              </xacro:unless>
+              <command_interface name="position"/>
               <state_interface name="position">
                 <param name="initial_value">${initial_positions['j1']}</param>
@@ -27,7 +25,5 @@
           </joint>
           <joint name="j2">
-              <xacro:unless value="${listen_only_mode}">
-                    <command_interface name="position"/>
-              </xacro:unless>
+              <command_interface name="position"/>
               <state_interface name="position">
                 <param name="initial_value">${initial_positions['j2']}</param>
@@ -35,7 +31,5 @@
           </joint>
           <joint name="j3">
-              <xacro:unless value="${listen_only_mode}">
-                    <command_interface name="position"/>
-              </xacro:unless>
+              <command_interface name="position"/>
               <state_interface name="position">
                 <param name="initial_value">${initial_positions['j3']}</param>
@@ -43,7 +37,5 @@
           </joint>
           <joint name="j4">
-              <xacro:unless value="${listen_only_mode}">
-                    <command_interface name="position"/>
-              </xacro:unless>
+              <command_interface name="position"/>
               <state_interface name="position">
                 <param name="initial_value">${initial_positions['j4']}</param>
@@ -51,19 +43,17 @@
           </joint>
           <joint name="j5">
-              <xacro:unless value="${listen_only_mode}">
-                    <command_interface name="position"/>
-              </xacro:unless>              <state_interface name="position">
+              <command_interface name="position"/>
+              <state_interface name="position">
                 <param name="initial_value">${initial_positions['j5']}</param>
               </state_interface>
           </joint>
           <joint name="j6">
-              <xacro:unless value="${listen_only_mode}">
-                    <command_interface name="position"/>
-              </xacro:unless>
-              <state_interface name="position">
+               <command_interface name="position"/>
+=              <state_interface name="position">
                 <param name="initial_value">${initial_positions['j6']}</param>
               </state_interface>
           </joint>
         </ros2_control>
+        </xacro:if>
         <xacro:if value="${ros2_control_header != 'world'}">
             <ros2_control name="${name}_rail" type="system">
@@ -122,5 +112,5 @@
         <xacro:if value="${control_system == 'gazebo'}">
             <gazebo>
-              <plugin filename="libign_ros2_control-system.so"
+              <plugin filename="libgz_ros2_control-system.so"
               name="gz_ros2_control::GazeboSimROS2ControlPlugin">
                   <parameters>$(find fairino10_v6_moveit2_config)/config/ros2_controllers.yaml</parameters>

File: src/fairino16_v6_moveit2_config/config/fairino16_v6_robot.ros2_control.xacro (robot description, xacro)
@@ -1,8 +1,9 @@
 <?xml version="1.0"?>
 <robot xmlns:xacro="http://www.ros.org/wiki/xacro">
-    <xacro:macro name="fairino16_v6_robot_ros2_control" params="name initial_positions_file ros2_control_header:=world control_system:=moveit gripper_name:=none gripper_hardware_connected:=false gripper_hardware_plugin:=none listen_only_mode:=true robot_ip_address:=192.168.58.2">
+    <xacro:macro name="fairino16_v6_robot_ros2_control" params="name initial_positions_file ros2_control_header:=world control_system:=moveit gripper_name:=none gripper_hardware_connected:=false gripper_hardware_plugin:=none listen_only_mode:=true robot_ip_address:=192.168.58.2 ">
         <xacro:property name="initial_positions" value="${xacro.load_yaml(initial_positions_file)['initial_positions']}"/>
         <!-- Xacro arg for control system (Defualted to Rviz/Moveit-->
         <xacro:property name="controllers_yaml_name" value="${'ros2_controllers.yaml' if ros2_control_header == 'world' else 'fairino16_' + ros2_control_header + '_ros2_controllers.yaml'}"/>
+        <xacro:if value="${str(listen_only_mode).lower() == 'false'}">
         <ros2_control name="${name}" type="system">
             <hardware>
@@ -12,5 +13,4 @@
               <xacro:if value="${control_system == 'hardware'}">
                   <plugin>fairino_hardware/FairinoHardwareInterface</plugin>
-                  <param name="robot_ip">${robot_ip_address}</param>
               </xacro:if>
               <xacro:if value="${control_system == 'gazebo'}">
@@ -19,7 +19,5 @@
           </hardware>
           <joint name="j1">
-              <xacro:unless value="${listen_only_mode}">
-                    <command_interface name="position"/>
-              </xacro:unless>
+              <command_interface name="position"/>
               <state_interface name="position">
                 <param name="initial_value">${initial_positions['j1']}</param>
@@ -27,7 +25,5 @@
           </joint>
           <joint name="j2">
-              <xacro:unless value="${listen_only_mode}">
-                    <command_interface name="position"/>
-              </xacro:unless>
+              <command_interface name="position"/>
               <state_interface name="position">
                 <param name="initial_value">${initial_positions['j2']}</param>
@@ -35,7 +31,5 @@
           </joint>
           <joint name="j3">
-              <xacro:unless value="${listen_only_mode}">
-                    <command_interface name="position"/>
-              </xacro:unless>
+              <command_interface name="position"/>
               <state_interface name="position">
                 <param name="initial_value">${initial_positions['j3']}</param>
@@ -43,7 +37,5 @@
           </joint>
           <joint name="j4">
-              <xacro:unless value="${listen_only_mode}">
-                    <command_interface name="position"/>
-              </xacro:unless>
+              <command_interface name="position"/>
               <state_interface name="position">
                 <param name="initial_value">${initial_positions['j4']}</param>
@@ -51,7 +43,5 @@
           </joint>
           <joint name="j5">
-              <xacro:unless value="${listen_only_mode}">
-                    <command_interface name="position"/>
-              </xacro:unless>
+              <command_interface name="position"/>
               <state_interface name="position">
                 <param name="initial_value">${initial_positions['j5']}</param>
@@ -59,12 +49,11 @@
           </joint>
           <joint name="j6">
-              <xacro:unless value="${listen_only_mode}">
-                    <command_interface name="position"/>
-              </xacro:unless>
-              <state_interface name="position">
+               <command_interface name="position"/>
+=              <state_interface name="position">
                 <param name="initial_value">${initial_positions['j6']}</param>
               </state_interface>
           </joint>
         </ros2_control>
+        </xacro:if>
         <xacro:if value="${ros2_control_header != 'world'}">
             <ros2_control name="${name}_rail" type="system">
@@ -123,5 +112,5 @@
         <xacro:if value="${control_system == 'gazebo'}">
             <gazebo>
-              <plugin filename="libign_ros2_control-system.so"
+              <plugin filename="libgz_ros2_control-system.so"
               name="gz_ros2_control::GazeboSimROS2ControlPlugin">
                   <parameters>$(find fairino16_v6_moveit2_config)/config/ros2_controllers.yaml</parameters>

File: src/fairino20_v6_moveit2_config/config/fairino20_v6_robot.ros2_control.xacro (robot description, xacro)
@@ -1,8 +1,9 @@
 <?xml version="1.0"?>
 <robot xmlns:xacro="http://www.ros.org/wiki/xacro">
-    <xacro:macro name="fairino20_v6_robot_ros2_control" params="name initial_positions_file ros2_control_header:=world control_system:=moveit gripper_name:=none gripper_hardware_connected:=false gripper_hardware_plugin:=mock_components/GenericSystem listen_only_mode:=true robot_ip_address:=192.168.58.2">
+    <xacro:macro name="fairino20_v6_robot_ros2_control" params="name initial_positions_file ros2_control_header:=world control_system:=moveit gripper_name:=none gripper_hardware_connected:=false gripper_hardware_plugin:=none listen_only_mode:=true robot_ip_address:=192.168.58.2 ">
         <xacro:property name="initial_positions" value="${xacro.load_yaml(initial_positions_file)['initial_positions']}"/>
         <!-- Xacro arg for control system (Defualted to Rviz/Moveit-->
         <xacro:property name="controllers_yaml_name" value="${'ros2_controllers.yaml' if ros2_control_header == 'world' else 'fairino20_' + ros2_control_header + '_ros2_controllers.yaml'}"/>
+        <xacro:if value="${str(listen_only_mode).lower() == 'false'}">
         <ros2_control name="${name}" type="system">
             <hardware>
@@ -12,5 +13,4 @@
               <xacro:if value="${control_system == 'hardware'}">
                   <plugin>fairino_hardware/FairinoHardwareInterface</plugin>
-                  <param name="robot_ip">${robot_ip_address}</param>
               </xacro:if>
               <xacro:if value="${control_system == 'gazebo'}">
@@ -19,7 +19,5 @@
           </hardware>
           <joint name="j1">
-              <xacro:unless value="${listen_only_mode}">
-                    <command_interface name="position"/>
-              </xacro:unless>
+              <command_interface name="position"/>
               <state_interface name="position">
                 <param name="initial_value">${initial_positions['j1']}</param>
@@ -27,7 +25,5 @@
           </joint>
           <joint name="j2">
-              <xacro:unless value="${listen_only_mode}">
-                    <command_interface name="position"/>
-              </xacro:unless>
+              <command_interface name="position"/>
               <state_interface name="position">
                 <param name="initial_value">${initial_positions['j2']}</param>
@@ -35,7 +31,5 @@
           </joint>
           <joint name="j3">
-              <xacro:unless value="${listen_only_mode}">
-                    <command_interface name="position"/>
-              </xacro:unless>
+              <command_interface name="position"/>
               <state_interface name="position">
                 <param name="initial_value">${initial_positions['j3']}</param>
@@ -43,7 +37,5 @@
           </joint>
           <joint name="j4">
-              <xacro:unless value="${listen_only_mode}">
-                    <command_interface name="position"/>
-              </xacro:unless>
+              <command_interface name="position"/>
               <state_interface name="position">
                 <param name="initial_value">${initial_positions['j4']}</param>
@@ -51,7 +43,5 @@
           </joint>
           <joint name="j5">
-              <xacro:unless value="${listen_only_mode}">
-                    <command_interface name="position"/>
-              </xacro:unless>
+              <command_interface name="position"/>
               <state_interface name="position">
                 <param name="initial_value">${initial_positions['j5']}</param>
@@ -59,12 +49,11 @@
           </joint>
           <joint name="j6">
-              <xacro:unless value="${listen_only_mode}">
-                    <command_interface name="position"/>
-              </xacro:unless>
-              <state_interface name="position">
+               <command_interface name="position"/>
+=              <state_interface name="position">
                 <param name="initial_value">${initial_positions['j6']}</param>
               </state_interface>
           </joint>
         </ros2_control>
+        </xacro:if>
         <xacro:if value="${ros2_control_header != 'world'}">
             <ros2_control name="${name}_rail" type="system">
@@ -123,5 +112,5 @@
         <xacro:if value="${control_system == 'gazebo'}">
             <gazebo>
-              <plugin filename="libign_ros2_control-system.so"
+              <plugin filename="libgz_ros2_control-system.so"
               name="gz_ros2_control::GazeboSimROS2ControlPlugin">
                   <parameters>$(find fairino20_v6_moveit2_config)/config/ros2_controllers.yaml</parameters>

File: src/fairino30_v6_moveit2_config/config/fairino30_v6_robot.ros2_control.xacro (robot description, xacro)
@@ -1,8 +1,9 @@
 <?xml version="1.0"?>
 <robot xmlns:xacro="http://www.ros.org/wiki/xacro">
-    <xacro:macro name="fairino30_v6_robot_ros2_control" params="name initial_positions_file ros2_control_header:=world control_system:=moveit gripper_name:=none gripper_hardware_connected:=false gripper_hardware_plugin:=mock_components/GenericSystem listen_only_mode:=true robot_ip_address:=192.168.58.2">
+    <xacro:macro name="fairino30_v6_robot_ros2_control" params="name initial_positions_file ros2_control_header:=world control_system:=moveit gripper_name:=none gripper_hardware_connected:=false gripper_hardware_plugin:=none listen_only_mode:=true robot_ip_address:=192.168.58.2 ">
         <xacro:property name="initial_positions" value="${xacro.load_yaml(initial_positions_file)['initial_positions']}"/>
         <!-- Xacro arg for control system (Defualted to Rviz/Moveit-->
         <xacro:property name="controllers_yaml_name" value="${'ros2_controllers.yaml' if ros2_control_header == 'world' else 'fairino30_' + ros2_control_header + '_ros2_controllers.yaml'}"/>
+        <xacro:if value="${str(listen_only_mode).lower() == 'false'}">
         <ros2_control name="${name}" type="system">
             <hardware>
@@ -18,7 +19,5 @@
           </hardware>
           <joint name="j1">
-              <xacro:unless value="${listen_only_mode}">
-                    <command_interface name="position"/>
-              </xacro:unless>
+              <command_interface name="position"/>
               <state_interface name="position">
                 <param name="initial_value">${initial_positions['j1']}</param>
@@ -26,7 +25,5 @@
           </joint>
           <joint name="j2">
-              <xacro:unless value="${listen_only_mode}">
-                    <command_interface name="position"/>
-              </xacro:unless>
+              <command_interface name="position"/>
               <state_interface name="position">
                 <param name="initial_value">${initial_positions['j2']}</param>
@@ -34,7 +31,5 @@
           </joint>
           <joint name="j3">
-              <xacro:unless value="${listen_only_mode}">
-                    <command_interface name="position"/>
-              </xacro:unless>
+              <command_interface name="position"/>
               <state_interface name="position">
                 <param name="initial_value">${initial_positions['j3']}</param>
@@ -42,7 +37,5 @@
           </joint>
           <joint name="j4">
-              <xacro:unless value="${listen_only_mode}">
-                    <command_interface name="position"/>
-              </xacro:unless>
+              <command_interface name="position"/>
               <state_interface name="position">
                 <param name="initial_value">${initial_positions['j4']}</param>
@@ -50,7 +43,5 @@
           </joint>
           <joint name="j5">
-              <xacro:unless value="${listen_only_mode}">
-                    <command_interface name="position"/>
-              </xacro:unless>
+              <command_interface name="position"/>
               <state_interface name="position">
                 <param name="initial_value">${initial_positions['j5']}</param>
@@ -58,12 +49,11 @@
           </joint>
           <joint name="j6">
-              <xacro:unless value="${listen_only_mode}">
-                    <command_interface name="position"/>
-              </xacro:unless>
-              <state_interface name="position">
+               <command_interface name="position"/>
+=              <state_interface name="position">
                 <param name="initial_value">${initial_positions['j6']}</param>
               </state_interface>
           </joint>
         </ros2_control>
+        </xacro:if>
         <xacro:if value="${ros2_control_header != 'world'}">
             <ros2_control name="${name}_rail" type="system">
@@ -122,5 +112,5 @@
         <xacro:if value="${control_system == 'gazebo'}">
             <gazebo>
-              <plugin filename="libign_ros2_control-system.so"
+              <plugin filename="libgz_ros2_control-system.so"
               name="gz_ros2_control::GazeboSimROS2ControlPlugin">
                   <parameters>$(find fairino30_v6_moveit2_config)/config/ros2_controllers.yaml</parameters>
